File: docs/lec2/schematics/schematics.kicad_sch (KiCad schematic)
At the start: 2 parts, among them U1 ESP-32S

Commit message: Updated material
Parts:
- removed U1: ESP-32S, BOARD, symbol ESP-32S:ESP-32S
- added ESP1: ~, symbol ESP-32S:ESP8266_dev
Connections:
- new net: ESP1. (USB), MPU1. (XDA) (x4)
- now unconnected: MPU1. (XDA), MPU1. (XDA), MPU1. (XDA)
Other:
- moved on the sheet: MPU1
Changed lines of the file:
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@@
 (kicad_sch (version 20230121) (generator eeschema)
   (paper "A4")
-  (wire (pts (xy 118.11 69.85) (xy 62.23 69.85))
+  (wire (pts (xy 71.12 91.44) (xy 71.12 137.16))
     (stroke (width 0) (type default))
   )
-  (wire (pts (xy 57.15 67.31) (xy 123.19 67.31))
+  (wire (pts (xy 91.44 107.95) (xy 91.44 144.78))
     (stroke (width 0) (type default))
   )
-  (wire (pts (xy 90.17 144.78) (xy 74.93 144.78))
+  (wire (pts (xy 91.44 144.78) (xy 118.11 144.78))
     (stroke (width 0) (type default))
   )
-  (wire (pts (xy 62.23 69.85) (xy 62.23 147.32))
+  (wire (pts (xy 71.12 137.16) (xy 118.11 137.16))
     (stroke (width 0) (type default))
   )
-  (wire (pts (xy 74.93 114.3) (xy 83.82 114.3))
+  (wire (pts (xy 93.98 91.44) (xy 71.12 91.44))
     (stroke (width 0) (type default))
   )
-  (wire (pts (xy 90.17 149.86) (xy 57.15 149.86))
+  (wire (pts (xy 83.82 104.14) (xy 83.82 142.24))
     (stroke (width 0) (type default))
   )
-  (wire (pts (xy 123.19 93.98) (xy 114.3 93.98))
+  (wire (pts (xy 93.98 95.25) (xy 74.93 95.25))
     (stroke (width 0) (type default))
   )
-  (wire (pts (xy 118.11 86.36) (xy 118.11 69.85))
+  (wire (pts (xy 74.93 139.7) (xy 118.11 139.7))
     (stroke (width 0) (type default))
   )
-  (wire (pts (xy 123.19 67.31) (xy 123.19 93.98))
+  (wire (pts (xy 74.93 95.25) (xy 74.93 139.7))
     (stroke (width 0) (type default))
   )
-  (wire (pts (xy 74.93 144.78) (xy 74.93 114.3))
+  (wire (pts (xy 93.98 107.95) (xy 91.44 107.95))
     (stroke (width 0) (type default))
   )
-  (wire (pts (xy 114.3 86.36) (xy 118.11 86.36))
+  (wire (pts (xy 93.98 104.14) (xy 83.82 104.14))
     (stroke (width 0) (type default))
   )
-  (wire (pts (xy 57.15 149.86) (xy 57.15 67.31))
+  (wire (pts (xy 83.82 142.24) (xy 118.11 142.24))
     (stroke (width 0) (type default))
   )
-  (wire (pts (xy 66.04 81.28) (xy 66.04 142.24))
-    (stroke (width 0) (type default))
-  )
-  (wire (pts (xy 83.82 81.28) (xy 66.04 81.28))
-    (stroke (width 0) (type default))
-  )
-  (wire (pts (xy 66.04 142.24) (xy 90.17 142.24))
-    (stroke (width 0) (type default))
-  )
-  (wire (pts (xy 62.23 147.32) (xy 90.17 147.32))
-    (stroke (width 0) (type default))
-  )
-  (symbol (lib_id "ESP-32S:ESP-32S") (at 99.06 104.14 0) (unit 1)
+  (symbol (lib_id "ESP-32S:ESP8266_dev") (at 102.87 88.9 0) (unit 1)
     (in_bom yes) (on_board yes) (dnp no) (fields_autoplaced)
-    (property "Reference" "U1" (at 99.06 74.93 0)
+    (property "Reference" "ESP1" (at 110.49 101.6 0)
+      (effects (font (size 1.27 1.27)) (justify left))
+    )
+    (property "Value" "~" (at 102.87 88.9 0)
+      (effects (font (size 1.27 1.27)))
+    )
+    (property "Footprint" "" (at 102.87 88.9 0)
       (effects (font (size 1.27 1.27)) hide)
     )
-    (property "Value" "ESP-32S" (at 99.06 77.47 0)
-      (effects (font (size 1.27 1.27)))
-    )
-    (property "Footprint" "BOARD" (at 99.06 104.14 0)
-      (effects (font (size 1.27 1.27)) (justify bottom) hide)
-    )
-    (property "Datasheet" "" (at 99.06 104.14 0)
+    (property "Datasheet" "" (at 102.87 88.9 0)
       (effects (font (size 1.27 1.27)) hide)
     )
-    (property "MAKER" "DarioBocc" (at 99.06 104.14 0)
-      (effects (font (size 1.27 1.27)) (justify bottom) hide)
-    )
-    (pin "1")
-    (pin "10")
-    (pin "11")
-    (pin "12")
-    (pin "13")
-    (pin "14")
-    (pin "15")
-    (pin "16")
-    (pin "17")
-    (pin "18")
-    (pin "19")
-    (pin "2")
-    (pin "20")
-    (pin "21")
-    (pin "22")
-    (pin "23")
-    (pin "24")
-    (pin "25")
-    (pin "26")
-    (pin "27")
-    (pin "28")
-    (pin "29")
-    (pin "3")
-    (pin "30")
-    (pin "31")
-    (pin "32")
-    (pin "33")
-    (pin "34")
-    (pin "35")
-    (pin "36")
-    (pin "37")
-    (pin "38")
-    (pin "4")
-    (pin "5")
-    (pin "6")
-    (pin "7")
-    (pin "8")
-    (pin "9")
+    (pin "")
+    (pin "")
+    (pin "")
+    (pin "")
+    (pin "")
     (instances
       (project "schematics"
         (path "/0ed7deae-b794-4414-a449-574f542852c6"
-          (reference "U1") (unit 1)
+          (reference "ESP1") (unit 1)
         )
       )
     )
   )
-  (symbol (lib_id "customlib:MPU-6050_Breakout_Board") (at 99.06 138.43 0) (unit 1)
+  (symbol (lib_id "customlib:MPU-6050_Breakout_Board") (at 127 133.35 0) (unit 1)
     (in_bom yes) (on_board no) (dnp no) (fields_autoplaced)
-    (property "Reference" "MPU1" (at 106.68 152.4 0)
+    (property "Reference" "MPU1" (at 134.62 147.32 0)
       (effects (font (size 1.27 1.27)) (justify left))
     )
-    (property "Value" "~" (at 99.06 138.43 0)
+    (property "Value" "~" (at 127 133.35 0)
       (effects (font (size 1.27 1.27)))
     )
-    (property "Footprint" "" (at 99.06 138.43 0)
+    (property "Footprint" "" (at 127 133.35 0)
       (effects (font (size 1.27 1.27)) hide)
     )
-    (property "Datasheet" "" (at 99.06 138.43 0)
+    (property "Datasheet" "" (at 127 133.35 0)
       (effects (font (size 1.27 1.27)) hide)
     )
